Commit message: Fix - Arrange xacro:property position in caster_wheel.xacro

File: xacro/caster_wheel.xacro (robot description, xacro)
@@ -1,6 +1,6 @@
 <?xml version="1.0"?>
 <robot xmlns:xacro="http://www.ros.org/wiki/xacro">
+    <xacro:property name="sphere_radius" value="0.0352" />
     <xacro:macro name="caster_wheel" params="prefix">
-        <xacro:property name="sphere_radius" value="0.0352" />
         <!-- Caster wheel -->
         <link name="${prefix}_caster_wheel_roll_link" >
