Commit message: Separate Gazebo colors and physical propeties from xacro file

File: xacro/barista_robot_model.urdf.xacro (robot description, xacro)
@@ -1,4 +1,5 @@
 <?xml version="1.0"?>
 <robot xmlns:xacro="http://www.ros.org/wiki/xacro" name="barista_robot">
+    <xacro:include filename="$(find barista_robot_description)/xacro/barista_robot_model.gazebo.xacro" />
     <xacro:include filename="$(find barista_robot_description)/xacro/drive_wheel.xacro" />
     <!-- Colors -->
@@ -15,4 +16,6 @@
         <color rgba="0.0 0.5 0.0 1"/>
     </material>
+    <!-- Gazebo physical properties and colors -->
+    <xacro:gazebo_elements />
     <!-- Base Link -->
     <link name="base_link">
@@ -34,27 +37,7 @@
         </inertial>
     </link>
-    <!-- Gazebo Color for Base link-->
-    <gazebo reference="base_link">
-        <material>Gazebo/Blue</material>
-    </gazebo>
     <!-- Drive Wheels -->
     <xacro:drive_wheel drive_wheel_name="left_drive_wheel" />
     <xacro:drive_wheel drive_wheel_name="right_drive_wheel" />
-    <!-- Gazebo - Left Drive Wheel -->
-    <gazebo reference="left_drive_wheel">
-        <material>Gazebo/Black</material>
-        <kp>1000000.0</kp>
-        <kd>100.0</kd>
-        <mu1>1.0</mu1>
-        <mu2>1.0</mu2>
-    </gazebo>
-    <!-- Gazebo - Right Drive Wheel -->
-    <gazebo reference="right_drive_wheel">
-        <material>Gazebo/Black</material>
-        <kp>1000000.0</kp>
-        <kd>100.0</kd>
-        <mu1>1.0</mu1>
-        <mu2>1.0</mu2>
-    </gazebo>
     <joint name="base_link_to_left_drive_wheel_joint" type="continuous">
         <origin rpy="0 0 0" xyz="0 0.126 -0.0775" />

Commit message: Macros added to urdf file to wrap some joints and dimensions

File: xacro/barista_robot_model.urdf.xacro (robot description, xacro)
@@ -8,4 +8,7 @@
     <xacro:include filename="$(find barista_robot_description)/xacro/cup_holder_tray.xacro" />
     <xacro:include filename="$(find barista_robot_description)/xacro/laser_scanner.xacro" />
+    <xacro:property name="base_link_radius" value="0.178" />
+    <xacro:property name="base_link_height" value="0.155" />
+    <xacro:property name="base_link_mass" value="0.5" />
     <!-- Colors -->
     <material name="blue">
@@ -21,4 +24,23 @@
         <color rgba="0.0 0.5 0.0 1"/>
     </material>
+    <!-- "cylinder_inertia"
+    # params="mass r l"
+    # mass: Mass in Kilograms of the link
+    # r: Radius of the cylinder in meters
+    # l: height of the cylinder in meters-->
+    <xacro:macro name="cylinder_inertia" params="mass r l" >
+        <inertia ixx="${mass*(3*r*r+l*l)/12}" ixy = "0" ixz = "0"
+                 iyy="${mass*(3*r*r+l*l)/12}" iyz = "0"
+                 izz="${mass*(r*r)/2}" />
+    </xacro:macro>
+    <!-- sphere_inertia"
+    # params="mass r"
+    # mass: Mass in Kilograms of the link
+    # r: Radius of the sphere in meters -->
+    <xacro:macro name="sphere_inertia" params="mass r" >
+        <inertia ixx="${2*mass*r*r/5}" ixy = "0" ixz = "0"
+                 iyy="${2*mass*r*r/5}" iyz = "0"
+                 izz="${2*mass*r*r/5}" />
+    </xacro:macro>
     <!-- Base Footprint -->
     <link name="base_footprint"/>
@@ -32,5 +54,5 @@
         <visual>
             <geometry>
-                <cylinder radius="0.178" length="0.155" />
+                <cylinder radius="${base_link_radius}" length="${base_link_height}" />
             </geometry>
             <material name="blue" />
@@ -38,11 +60,12 @@
         <collision>
             <geometry>
-                <cylinder radius="0.178" length="0.155" />
+                <cylinder radius="${base_link_radius}" length="${base_link_height}" />
             </geometry>
         </collision>
         <inertial>
-            <mass value="0.5" />
+            <mass value="${base_link_mass}" />
             <origin rpy="0 0 0" xyz="0 0 0" />
-            <inertia ixx="0.0049615416667" ixy="0" ixz="0" iyy="0.0049615416667" iyz="0" izz="0.007921" />
+            <xacro:cylinder_inertia mass="${base_link_mass}" r="${base_link_radius}" l="${base_link_height}" />
+            <!--inertia ixx="0.0049615416667" ixy="0" ixz="0" iyy="0.0049615416667" iyz="0" izz="0.007921" /-->
         </inertial>
     </link>
@@ -51,5 +74,5 @@
     <xacro:drive_wheel drive_wheel_name="right_drive_wheel" />
     <joint name="base_link_to_left_drive_wheel_joint" type="continuous">
-        <origin rpy="0 0 0" xyz="0 0.126 -0.0775" />
+        <origin rpy="0 0 0" xyz="0 0.126 -${base_link_height}/2" />
         <parent link="base_link" />
         <child link="left_drive_wheel" />
@@ -57,13 +80,13 @@
     </joint>
     <joint name="base_link_to_right_drive_wheel_joint" type="continuous">
-        <origin rpy="0 0 0" xyz="0 -0.126 -0.0775" />
+        <origin rpy="0 0 0" xyz="0 -0.126 -${base_link_height}/2" />
         <parent link="base_link" />
         <child link="right_drive_wheel" />
         <axis xyz="0 1 0" />
     </joint>
-    <!-- Caster Wheels -->
+    <!-- Caster Wheels + Joints-->
     <xacro:caster_wheel prefix="front" />
     <xacro:caster_wheel prefix="back" />
-    <joint name="front_caster_wheel_roll_joint" type="continuous" >
+    <!--joint name="front_caster_wheel_roll_joint" type="continuous" >
         <origin rpy="0 0 0" xyz="0.11 0 -0.0775" />
         <parent link="base_link" />
@@ -100,5 +123,5 @@
         <child link="back_caster_wheel_yaw_link" />
         <axis xyz="0 0 1" />
-    </joint>
+    </joint-->
     <!-- Standoff rods -->
     <xacro:standoff_rod prefix="upper_right" />
@@ -138,5 +161,5 @@
         <xacro:laser_scanner />
         <joint name="base_link_to_laser_scan_link_joint" type="fixed">
-            <origin rpy="0 0 0" xyz="0.089 0 0.0775"/>
+            <origin rpy="0 0 0" xyz="0.089 0 ${base_link_height}/2"/>
             <parent link="base_link" />
             <child link="laser_scan_link" />

File: xacro/caster_wheel.xacro (robot description, xacro)
@@ -1,19 +1,32 @@
 <?xml version="1.0"?>
 <robot xmlns:xacro="http://www.ros.org/wiki/xacro">
-    <xacro:property name="sphere_radius" value="0.0352" />
+    <xacro:property name="caster_wheel_radius" value="0.0352" />
+    <xacro:property name="caster_wheel_mass" value="0.05" />
+    <xacro:property name="negligible_mass" value="0.001" />
+    <!-- sphere_inertia"
+    # params="mass r"
+    # mass: Mass in Kilograms of the link
+    # r: Radius of the sphere in meters -->
+    <xacro:macro name="sphere_inertia" params="mass r" >
+        <inertia ixx="${2*mass*r*r/5}" ixy = "0" ixz = "0"
+                 iyy="${2*mass*r*r/5}" iyz = "0"
+                 izz="${2*mass*r*r/5}" />
+    </xacro:macro>
     <xacro:macro name="caster_wheel" params="prefix">
         <!-- Caster wheel -->
         <link name="${prefix}_caster_wheel_roll_link" >
             <inertial>
-                <mass value="0.001" />
+                <mass value="${negligible_mass}" />
                 <origin rpy="0 0 0" xyz="0 0 0"/>
-                <inertia ixx="0.000000495616" ixy="0" ixz="0" iyy="0.000000495616" iyz="0" izz="0.000000495616" />
+                <xacro:sphere_inertia mass="${negligible_mass}" r="${caster_wheel_radius}" />
+                <!--inertia ixx="0.000000495616" ixy="0" ixz="0" iyy="0.000000495616" iyz="0" izz="0.000000495616" /-->
             </inertial>
         </link>
         <link name="${prefix}_caster_wheel_pitch_link" >
             <inertial>
-                <mass value="0.001" />
+                <mass value="${negligible_mass}" />
                 <origin rpy="0 0 0" xyz="0 0 0"/>
-                <inertia ixx="0.000000495616" ixy="0" ixz="0" iyy="0.000000495616" iyz="0" izz="0.000000495616" />
+                <xacro:sphere_inertia mass="${negligible_mass}" r="${caster_wheel_radius}" />
+                <!--inertia ixx="0.000000495616" ixy="0" ixz="0" iyy="0.000000495616" iyz="0" izz="0.000000495616" /-->
             </inertial>
         </link>
@@ -21,5 +34,5 @@
             <visual>
                 <geometry>
-                    <sphere radius="${sphere_radius}" />
+                    <sphere radius="${caster_wheel_radius}" />
                 </geometry>
                 <material name="green_dark" />
@@ -27,13 +40,32 @@
             <collision>
                 <geometry>
-                    <sphere radius="${sphere_radius}" />
+                    <sphere radius="${caster_wheel_radius}" />
                 </geometry>
             </collision>
             <inertial>
-                <mass value="0.05" />
+                <mass value="${caster_wheel_mass}" />
                 <origin rpy="0 0 0" xyz="0 0 0"/>
-                <inertia ixx="0.0000247808" ixy="0" ixz="0" iyy="0.0000247808" iyz="0" izz="0.0000247808" />
+                <xacro:sphere_inertia mass="${caster_wheel_mass}" r="${caster_wheel_radius}" />
+                <!--inertia ixx="0.0000247808" ixy="0" ixz="0" iyy="0.0000247808" iyz="0" izz="0.0000247808" /-->
             </inertial>
         </link>
+        <joint name="${prefix}_caster_wheel_roll_joint" type="continuous" >
+            <origin rpy="0 0 0" xyz="0.11 0 -0.0775" />
+            <parent link="base_link" />
+            <child link="${prefix}_caster_wheel_roll_link" />
+            <axis xyz="1 0 0" />
+        </joint>
+        <joint name="${prefix}_caster_wheel_pitch_joint" type="continuous" >
+            <origin rpy="0 0 0" xyz="0 0 0" />
+            <parent link="${prefix}_caster_wheel_roll_link" />
+            <child link="${prefix}_caster_wheel_pitch_link" />
+            <axis xyz="0 1 0" />
+        </joint>
+        <joint name="${prefix}_caster_wheel_yaw_joint" type="continuous" >
+            <origin rpy="0 0 0" xyz="0 0 0" />
+            <parent link="${prefix}_caster_wheel_pitch_link" />
+            <child link="${prefix}_caster_wheel_yaw_link" />
+            <axis xyz="0 0 1" />
+        </joint>
     </xacro:macro>
 </robot>

File: xacro/cup_holder_tray.xacro (robot description, xacro)
@@ -3,4 +3,15 @@
     <xacro:property name="tray_radius" value="0.160" />
     <xacro:property name="tray_width" value="0.090" />
+    <xacro:property name="tray_mass" value="0.25" />
+    <!-- "cylinder_inertia"
+    # params="mass r l"
+    # mass: Mass in Kilograms of the link
+    # r: Radius of the cylinder in meters
+    # l: height of the cylinder in meters-->
+    <xacro:macro name="cylinder_inertia" params="mass r l" >
+        <inertia ixx="${mass*(3*r*r+l*l)/12}" ixy = "0" ixz = "0"
+                 iyy="${mass*(3*r*r+l*l)/12}" iyz = "0"
+                 izz="${mass*(r*r)/2}" />
+    </xacro:macro>
     <xacro:macro name="cup_holder_tray">
         <!-- Cup Holder Tray -->
@@ -18,7 +29,8 @@
             </collision>
             <inertial>
-                <mass value="0.25" />
+                <mass value="${tray_mass}" />
                 <origin rpy="0 0 0" xyz="0 0 0" />
-                <inertia ixx="0.00176875" ixy="0" ixz="0" iyy="0.00176875" iyz="0" izz="0.0032" />
+                <xacro:cylinder_inertia mass="${tray_mass}" r="${tray_radius}" l="${tray_width}" />
+                <!--inertia ixx="0.00176875" ixy="0" ixz="0" iyy="0.00176875" iyz="0" izz="0.0032" /-->
             </inertial>
         </link>

File: xacro/drive_wheel.xacro (robot description, xacro)
@@ -3,4 +3,15 @@
     <xacro:property name="drive_wheel_radius" value="0.0352"/>
     <xacro:property name="drive_wheel_width" value="0.0206"/>
+    <xacro:property name="drive_wheel_mass" value="0.05"/>
+    <!-- "cylinder_inertia"
+    # params="mass r l"
+    # mass: Mass in Kilograms of the link
+    # r: Radius of the cylinder in meters
+    # l: height of the cylinder in meters-->
+    <xacro:macro name="cylinder_inertia" params="mass r l" >
+        <inertia ixx="${mass*(3*r*r+l*l)/12}" ixy = "0" ixz = "0"
+                 iyy="${mass*(3*r*r+l*l)/12}" iyz = "0"
+                 izz="${mass*(r*r)/2}" />
+    </xacro:macro>
     <xacro:macro name="drive_wheel" params="drive_wheel_name">
         <!-- Drive Wheel -->
@@ -20,7 +31,8 @@
             </collision>
             <inertial>
-                <mass value="0.05" />
+                <mass value="${drive_wheel_mass}" />
                 <origin rpy="0 0 0" xyz="0 0 0" />
-                <inertia ixx="0.0000172561667" ixy="0" ixz="0" iyy="0.0000172561667" iyz="0" izz="0.000030976" />
+                <xacro:cylinder_inertia mass="${drive_wheel_mass}" r="${drive_wheel_radius}" l="${drive_wheel_width}" />
+                <!--inertia ixx="0.0000172561667" ixy="0" ixz="0" iyy="0.0000172561667" iyz="0" izz="0.000030976" /-->
             </inertial>
         </link>

File: xacro/laser_scanner.xacro (robot description, xacro)
@@ -1,4 +1,17 @@
 <?xml version="1.0"?>
 <robot xmlns:xacro="http://www.ros.org/wiki/xacro">
+    <xacro:property name="box_x_size" value="0.2" />
+    <xacro:property name="box_y_size" value="0.2" />
+    <xacro:property name="box_z_size" value="0.5" />
+    <xacro:property name="box_mass" value="0.05" />
+    <!-- "box_inertia"
+    # params="mass x y z"
+    # mass: Mass in Kilograms of the link
+    # x,y,z: Are the size of each side of the box in each of the axes in meters -->
+    <xacro:macro name="box_inertia" params="mass x y z" >
+        <inertia ixx="${mass*(y*y+z*z)/12}" ixy = "0" ixz = "0"
+                 iyy="${mass*(x*x+z*z)/12}" iyz = "0"
+                 izz="${mass*(x*x+z*z)/12}" />
+    </xacro:macro>
     <xacro:macro name="laser_scanner">
         <!-- Laser Scan (Model) -->
@@ -11,11 +24,12 @@
             <collision>
                 <geometry>
-                    <box size="0.02 0.02 0.05" />
+                    <box size="${box_x_size} ${box_y_size} ${box_z_size}" />
                 </geometry>
             </collision>
             <inertial>
-                <mass value="0.05" />
+                <mass value="${box_mass}" />
                 <origin rpy="0 0 0" xyz="0 0 0" />
-                <inertia ixx="0.0000110833333" ixy="0" ixz="0" iyy="0.0000110833333" iyz="0" izz="0.0000033333333" />
+                <xacro:box_inertia mass="${box_mass}" x="${box_x_size}" y="${box_y_size}" z="${box_z_size}" />
+                <!--inertia ixx="0.0000110833333" ixy="0" ixz="0" iyy="0.0000110833333" iyz="0" izz="0.0000033333333" /-->
             </inertial>
         </link>

File: xacro/standoff_rod.xacro (robot description, xacro)
@@ -3,4 +3,15 @@
     <xacro:property name="rod_radius" value="0.01" />
     <xacro:property name="rod_height" value="0.22" />
+    <xacro:property name="rod_mass" value="0.025" />
+    <!-- "cylinder_inertia"
+    # params="mass r l"
+    # mass: Mass in Kilograms of the link
+    # r: Radius of the cylinder in meters
+    # l: height of the cylinder in meters-->
+    <xacro:macro name="cylinder_inertia" params="mass r l" >
+        <inertia ixx="${mass*(3*r*r+l*l)/12}" ixy = "0" ixz = "0"
+                 iyy="${mass*(3*r*r+l*l)/12}" iyz = "0"
+                 izz="${mass*(r*r)/2}" />
+    </xacro:macro>
     <xacro:macro name="standoff_rod" params="prefix">
         <!-- Standoff rod -->
@@ -18,7 +29,8 @@
             </collision>
             <inertial>
-                <mass value="0.025" />
+                <mass value="${rod_mass}" />
                 <origin rpy="0 0 0" xyz="0 0 0" />
-                <inertia ixx="0.0001014583333" ixy="0" ixz="0" iyy="0.0001014583333" iyz="0" izz="0.00000125" />
+                <xacro:cylinder_inertia mass="${rod_mass}" r="${rod_radius}" l="${rod_height}" />
+                <!--inertia ixx="0.0001014583333" ixy="0" ixz="0" iyy="0.0001014583333" iyz="0" izz="0.00000125" /-->
             </inertial>
         </link>
