Commit message: Update macros in xacro files to create the associate joint to the link + Update main xacro

File: xacro/barista_robot_model.urdf.xacro (robot description, xacro)
@@ -11,4 +11,5 @@
     <xacro:property name="base_link_height" value="0.155" />
     <xacro:property name="base_link_mass" value="0.5" />
+    <xacro:property name="drive_wheel_radius" value="0.0352"/>
     <!-- Colors -->
     <material name="blue">
@@ -34,17 +35,8 @@
                  izz="${mass*(r*r)/2}" />
     </xacro:macro>
-    <!-- sphere_inertia"
-    # params="mass r"
-    # mass: Mass in Kilograms of the link
-    # r: Radius of the sphere in meters -->
-    <xacro:macro name="sphere_inertia" params="mass r" >
-        <inertia ixx="${2*mass*r*r/5}" ixy = "0" ixz = "0"
-                 iyy="${2*mass*r*r/5}" iyz = "0"
-                 izz="${2*mass*r*r/5}" />
-    </xacro:macro>
     <!-- Base Footprint -->
     <link name="base_footprint"/>
     <joint name="base_footprint_to_base_link" type="fixed">
-        <origin rpy="0 0 0" xyz="0 0 0.1127" />
+        <origin rpy="0 0 0" xyz="0 0 ${base_link_height/2 + drive_wheel_radius}" />
         <parent link="base_footprint"/>
         <child link="base_link"/>
@@ -71,89 +63,17 @@
     </link>
     <!-- Drive Wheels -->
-    <xacro:drive_wheel drive_wheel_name="left_drive_wheel" />
-    <xacro:drive_wheel drive_wheel_name="right_drive_wheel" />
-    <joint name="base_link_to_left_drive_wheel_joint" type="continuous">
-        <origin rpy="0 0 0" xyz="0 0.126 -${base_link_height}/2" />
-        <parent link="base_link" />
-        <child link="left_drive_wheel" />
-        <axis xyz="0 1 0" />
-    </joint>
-    <joint name="base_link_to_right_drive_wheel_joint" type="continuous">
-        <origin rpy="0 0 0" xyz="0 -0.126 -${base_link_height}/2" />
-        <parent link="base_link" />
-        <child link="right_drive_wheel" />
-        <axis xyz="0 1 0" />
-    </joint>
+    <xacro:drive_wheel drive_wheel_name="left_drive_wheel" origin_joint_y="0.126"/>
+    <xacro:drive_wheel drive_wheel_name="right_drive_wheel" origin_joint_y="-0.126" />
     <!-- Caster Wheels + Joints-->
-    <xacro:caster_wheel prefix="front" />
-    <xacro:caster_wheel prefix="back" />
-    <!--joint name="front_caster_wheel_roll_joint" type="continuous" >
-        <origin rpy="0 0 0" xyz="0.11 0 -0.0775" />
-        <parent link="base_link" />
-        <child link="front_caster_wheel_roll_link" />
-        <axis xyz="1 0 0" />
-    </joint>
-    <joint name="front_caster_wheel_pitch_joint" type="continuous" >
-        <origin rpy="0 0 0" xyz="0 0 0" />
-        <parent link="front_caster_wheel_roll_link" />
-        <child link="front_caster_wheel_pitch_link" />
-        <axis xyz="0 1 0" />
-    </joint>
-    <joint name="front_caster_wheel_yaw_joint" type="continuous" >
-        <origin rpy="0 0 0" xyz="0 0 0" />
-        <parent link="front_caster_wheel_pitch_link" />
-        <child link="front_caster_wheel_yaw_link" />
-        <axis xyz="0 0 1" />
-    </joint>
-    <joint name="back_caster_wheel_roll_joint" type="continuous" >
-        <origin rpy="0 0 0" xyz="-0.11 0 -0.0775" />
-        <parent link="base_link" />
-        <child link="back_caster_wheel_roll_link" />
-        <axis xyz="1 0 0" />
-    </joint>
-    <joint name="back_caster_wheel_pitch_joint" type="continuous" >
-        <origin rpy="0 0 0" xyz="0 0 0" />
-        <parent link="back_caster_wheel_roll_link" />
-        <child link="back_caster_wheel_pitch_link" />
-        <axis xyz="0 1 0" />
-    </joint>
-    <joint name="back_caster_wheel_yaw_joint" type="continuous" >
-        <origin rpy="0 0 0" xyz="0 0 0" />
-        <parent link="back_caster_wheel_pitch_link" />
-        <child link="back_caster_wheel_yaw_link" />
-        <axis xyz="0 0 1" />
-    </joint-->
+    <xacro:caster_wheel prefix="front" joint_origin_x="0.11" />
+    <xacro:caster_wheel prefix="back" joint_origin_x="-0.11" />
     <!-- Standoff rods -->
-    <xacro:standoff_rod prefix="upper_right" />
-    <xacro:standoff_rod prefix="lower_right" />
-    <xacro:standoff_rod prefix="upper_left" />
-    <xacro:standoff_rod prefix="lower_left" />
-    <joint name="base_link_to_upper_right_rod_joint" type="fixed" >
-        <origin rpy="0 0 0" xyz="0.07 -0.11 0.1875" />
-        <parent link="base_link" />
-        <child link="upper_right_rod" />
-    </joint>
-    <joint name="base_link_to_lower_right_rod_joint" type="fixed" >
-        <origin rpy="0 0 0" xyz="-0.07 -0.11 0.1875" />
-        <parent link="base_link" />
-        <child link="lower_right_rod" />
-    </joint>
-    <joint name="base_link_to_lower_left_rod_joint" type="fixed" >
-        <origin rpy="0 0 0" xyz="-0.07 0.11 0.1875" />
-        <parent link="base_link" />
-        <child link="lower_left_rod" />
-    </joint>
-     <joint name="base_link_to_upper_left_rod_joint" type="fixed" >
-        <origin rpy="0 0 0" xyz="0.07 0.11 0.1875" />
-        <parent link="base_link" />
-        <child link="upper_left_rod" />
-    </joint>
+    <xacro:standoff_rod prefix="upper_right" origin_joint_x="0.07" origin_joint_y="-0.11" />
+    <xacro:standoff_rod prefix="lower_right" origin_joint_x="-0.07" origin_joint_y="-0.11" />
+    <xacro:standoff_rod prefix="lower_left" origin_joint_x="-0.07" origin_joint_y="0.11" />
+    <xacro:standoff_rod prefix="upper_left" origin_joint_x="0.07" origin_joint_y="0.11" />
     <!-- Cup Holder Tray -->
     <xacro:cup_holder_tray />
-    <joint name="base_link_to_cup_holder_tray_joint" type="fixed">
-        <origin rpy="0 0 0" xyz="0 0 0.3425" />
-        <parent link="base_link" />
-        <child link="cup_holder_tray" />
-    </joint>
+    <!-- Include Laser scanner or not -->
     <xacro:arg name="include_laser" default="true"/>
     <xacro:if value="$(arg include_laser)">
@@ -161,5 +81,5 @@
         <xacro:laser_scanner />
         <joint name="base_link_to_laser_scan_link_joint" type="fixed">
-            <origin rpy="0 0 0" xyz="0.089 0 ${base_link_height}/2"/>
+            <origin rpy="0 0 0" xyz="0.089 0 ${base_link_height/2}"/>
             <parent link="base_link" />
             <child link="laser_scan_link" />

File: xacro/caster_wheel.xacro (robot description, xacro)
@@ -13,5 +13,5 @@
                  izz="${2*mass*r*r/5}" />
     </xacro:macro>
-    <xacro:macro name="caster_wheel" params="prefix">
+    <xacro:macro name="caster_wheel" params="prefix joint_origin_x">
         <!-- Caster wheel -->
         <link name="${prefix}_caster_wheel_roll_link" >
@@ -51,5 +51,5 @@
         </link>
         <joint name="${prefix}_caster_wheel_roll_joint" type="continuous" >
-            <origin rpy="0 0 0" xyz="0.11 0 -0.0775" />
+            <origin rpy="0 0 0" xyz="${joint_origin_x} 0 -0.0775" />
             <parent link="base_link" />
             <child link="${prefix}_caster_wheel_roll_link" />

File: xacro/cup_holder_tray.xacro (robot description, xacro)
@@ -35,4 +35,9 @@
             </inertial>
         </link>
+        <joint name="base_link_to_cup_holder_tray_joint" type="fixed">
+            <origin rpy="0 0 0" xyz="0 0 0.3425" />
+            <parent link="base_link" />
+            <child link="cup_holder_tray" />
+        </joint>
     </xacro:macro>
 </robot>

File: xacro/drive_wheel.xacro (robot description, xacro)
@@ -4,4 +4,5 @@
     <xacro:property name="drive_wheel_width" value="0.0206"/>
     <xacro:property name="drive_wheel_mass" value="0.05"/>
+    <xacro:property name="base_link_height" value="0.155" />
     <!-- "cylinder_inertia"
     # params="mass r l"
@@ -14,5 +15,5 @@
                  izz="${mass*(r*r)/2}" />
     </xacro:macro>
-    <xacro:macro name="drive_wheel" params="drive_wheel_name">
+    <xacro:macro name="drive_wheel" params="drive_wheel_name origin_joint_y">
         <!-- Drive Wheel -->
         <link name="${drive_wheel_name}">
@@ -37,4 +38,10 @@
             </inertial>
         </link>
+        <joint name="base_link_to_${drive_wheel_name}_joint" type="continuous">
+            <origin rpy="0 0 0" xyz="0 ${origin_joint_y} ${-base_link_height/2}" />
+            <parent link="base_link" />
+            <child link="${drive_wheel_name}" />
+            <axis xyz="0 1 0" />
+        </joint>
     </xacro:macro>
 </robot>

File: xacro/laser_scanner.xacro (robot description, xacro)
@@ -1,7 +1,7 @@
 <?xml version="1.0"?>
 <robot xmlns:xacro="http://www.ros.org/wiki/xacro">
-    <xacro:property name="box_x_size" value="0.2" />
-    <xacro:property name="box_y_size" value="0.2" />
-    <xacro:property name="box_z_size" value="0.5" />
+    <xacro:property name="box_x_size" value="0.02" />
+    <xacro:property name="box_y_size" value="0.02" />
+    <xacro:property name="box_z_size" value="0.05" />
     <xacro:property name="box_mass" value="0.05" />
     <!-- "box_inertia"

File: xacro/standoff_rod.xacro (robot description, xacro)
@@ -14,5 +14,5 @@
                  izz="${mass*(r*r)/2}" />
     </xacro:macro>
-    <xacro:macro name="standoff_rod" params="prefix">
+    <xacro:macro name="standoff_rod" params="prefix origin_joint_x origin_joint_y">
         <!-- Standoff rod -->
         <link name="${prefix}_rod" >
@@ -35,4 +35,9 @@
             </inertial>
         </link>
+        <joint name="base_link_to_${prefix}_rod_joint" type="fixed" >
+            <origin rpy="0 0 0" xyz="${origin_joint_x} ${origin_joint_y} 0.1875" />
+            <parent link="base_link" />
+            <child link="${prefix}_rod" />
+        </joint>
     </xacro:macro>
 </robot>

Commit message: Gather all xacro:property to the main xacro file

File: xacro/barista_robot_model.urdf.xacro (robot description, xacro)
@@ -8,8 +8,24 @@
     <xacro:include filename="$(find barista_robot_description)/xacro/cup_holder_tray.xacro" />
     <xacro:include filename="$(find barista_robot_description)/xacro/laser_scanner.xacro" />
+    <!-- Robot global dimensions -->
     <xacro:property name="base_link_radius" value="0.178" />
     <xacro:property name="base_link_height" value="0.155" />
     <xacro:property name="base_link_mass" value="0.5" />
     <xacro:property name="drive_wheel_radius" value="0.0352"/>
+    <xacro:property name="drive_wheel_width" value="0.0206"/>
+    <xacro:property name="drive_wheel_mass" value="0.05"/>
+    <xacro:property name="caster_wheel_radius" value="0.0352" />
+    <xacro:property name="caster_wheel_mass" value="0.05" />
+    <xacro:property name="negligible_mass" value="0.001" />
+    <xacro:property name="rod_radius" value="0.01" />
+    <xacro:property name="rod_height" value="0.22" />
+    <xacro:property name="rod_mass" value="0.025" />
+    <xacro:property name="tray_radius" value="0.160" />
+    <xacro:property name="tray_width" value="0.090" />
+    <xacro:property name="tray_mass" value="0.25" />
+    <xacro:property name="box_x_size" value="0.02" /> <!-- Laser scanner -->
+    <xacro:property name="box_y_size" value="0.02" />
+    <xacro:property name="box_z_size" value="0.05" />
+    <xacro:property name="box_mass" value="0.05" />
     <!-- Colors -->
     <material name="blue">

File: xacro/caster_wheel.xacro (robot description, xacro)
@@ -1,7 +1,7 @@
 <?xml version="1.0"?>
 <robot xmlns:xacro="http://www.ros.org/wiki/xacro">
-    <xacro:property name="caster_wheel_radius" value="0.0352" />
+    <!--xacro:property name="caster_wheel_radius" value="0.0352" />
     <xacro:property name="caster_wheel_mass" value="0.05" />
-    <xacro:property name="negligible_mass" value="0.001" />
+    <xacro:property name="negligible_mass" value="0.001" /-->
     <!-- sphere_inertia"
     # params="mass r"

File: xacro/cup_holder_tray.xacro (robot description, xacro)
@@ -1,7 +1,4 @@
 <?xml version="1.0"?>
 <robot xmlns:xacro="http://www.ros.org/wiki/xacro">
-    <xacro:property name="tray_radius" value="0.160" />
-    <xacro:property name="tray_width" value="0.090" />
-    <xacro:property name="tray_mass" value="0.25" />
     <!-- "cylinder_inertia"
     # params="mass r l"

File: xacro/drive_wheel.xacro (robot description, xacro)
@@ -1,8 +1,4 @@
 <?xml version="1.0"?>
 <robot xmlns:xacro="http://www.ros.org/wiki/xacro">
-    <xacro:property name="drive_wheel_radius" value="0.0352"/>
-    <xacro:property name="drive_wheel_width" value="0.0206"/>
-    <xacro:property name="drive_wheel_mass" value="0.05"/>
-    <xacro:property name="base_link_height" value="0.155" />
     <!-- "cylinder_inertia"
     # params="mass r l"

File: xacro/laser_scanner.xacro (robot description, xacro)
@@ -1,8 +1,4 @@
 <?xml version="1.0"?>
 <robot xmlns:xacro="http://www.ros.org/wiki/xacro">
-    <xacro:property name="box_x_size" value="0.02" />
-    <xacro:property name="box_y_size" value="0.02" />
-    <xacro:property name="box_z_size" value="0.05" />
-    <xacro:property name="box_mass" value="0.05" />
     <!-- "box_inertia"
     # params="mass x y z"

File: xacro/standoff_rod.xacro (robot description, xacro)
@@ -1,7 +1,4 @@
 <?xml version="1.0"?>
 <robot xmlns:xacro="http://www.ros.org/wiki/xacro">
-    <xacro:property name="rod_radius" value="0.01" />
-    <xacro:property name="rod_height" value="0.22" />
-    <xacro:property name="rod_mass" value="0.025" />
     <!-- "cylinder_inertia"
     # params="mass r l"

Commit message: Gathered inertia macros into a single file and included this file to all needed xacro files

File: xacro/barista_robot_model.urdf.xacro (robot description, xacro)
@@ -1,11 +1,4 @@
 <?xml version="1.0"?>
 <robot xmlns:xacro="http://www.ros.org/wiki/xacro" name="barista_robot">
-    <xacro:include filename="$(find barista_robot_description)/xacro/barista_robot_model.gazebo.xacro" />
-    <xacro:include filename="$(find barista_robot_description)/xacro/barista_robot_model.gazebo_plugins.xacro" />
-    <xacro:include filename="$(find barista_robot_description)/xacro/drive_wheel.xacro" />
-    <xacro:include filename="$(find barista_robot_description)/xacro/caster_wheel.xacro" />
-    <xacro:include filename="$(find barista_robot_description)/xacro/standoff_rod.xacro" />
-    <xacro:include filename="$(find barista_robot_description)/xacro/cup_holder_tray.xacro" />
-    <xacro:include filename="$(find barista_robot_description)/xacro/laser_scanner.xacro" />
     <!-- Robot global dimensions -->
     <xacro:property name="base_link_radius" value="0.178" />
@@ -25,7 +18,15 @@
     <xacro:property name="tray_mass" value="0.25" />
     <xacro:property name="box_x_size" value="0.02" /> <!-- Laser scanner -->
-    <xacro:property name="box_y_size" value="0.02" />
-    <xacro:property name="box_z_size" value="0.05" />
-    <xacro:property name="box_mass" value="0.05" />
+    <xacro:property name="box_y_size" value="0.02" /> <!-- Laser scanner -->
+    <xacro:property name="box_z_size" value="0.05" /> <!-- Laser scanner -->
+    <xacro:property name="box_mass" value="0.05" />   <!-- Laser scanner -->
+    <!-- Included Macros  -->
+    <xacro:include filename="$(find barista_robot_description)/xacro/barista_robot_model.gazebo.xacro" />
+    <xacro:include filename="$(find barista_robot_description)/xacro/barista_robot_model.gazebo_plugins.xacro" />
+    <xacro:include filename="$(find barista_robot_description)/xacro/drive_wheel.xacro" />
+    <xacro:include filename="$(find barista_robot_description)/xacro/caster_wheel.xacro" />
+    <xacro:include filename="$(find barista_robot_description)/xacro/standoff_rod.xacro" />
+    <xacro:include filename="$(find barista_robot_description)/xacro/cup_holder_tray.xacro" />
+    <xacro:include filename="$(find barista_robot_description)/xacro/laser_scanner.xacro" />
     <!-- Colors -->
     <material name="blue">
@@ -41,14 +42,4 @@
         <color rgba="0.0 0.5 0.0 1"/>
     </material>
-    <!-- "cylinder_inertia"
-    # params="mass r l"
-    # mass: Mass in Kilograms of the link
-    # r: Radius of the cylinder in meters
-    # l: height of the cylinder in meters-->
-    <xacro:macro name="cylinder_inertia" params="mass r l" >
-        <inertia ixx="${mass*(3*r*r+l*l)/12}" ixy = "0" ixz = "0"
-                 iyy="${mass*(3*r*r+l*l)/12}" iyz = "0"
-                 izz="${mass*(r*r)/2}" />
-    </xacro:macro>
     <!-- Base Footprint -->
     <link name="base_footprint"/>
@@ -78,5 +69,5 @@
         </inertial>
     </link>
-    <!-- Drive Wheels -->
+    <!-- Drive Wheels + Joints -->
     <xacro:drive_wheel drive_wheel_name="left_drive_wheel" origin_joint_y="0.126"/>
     <xacro:drive_wheel drive_wheel_name="right_drive_wheel" origin_joint_y="-0.126" />
@@ -84,10 +75,10 @@
     <xacro:caster_wheel prefix="front" joint_origin_x="0.11" />
     <xacro:caster_wheel prefix="back" joint_origin_x="-0.11" />
-    <!-- Standoff rods -->
+    <!-- Standoff rods + Joints -->
     <xacro:standoff_rod prefix="upper_right" origin_joint_x="0.07" origin_joint_y="-0.11" />
     <xacro:standoff_rod prefix="lower_right" origin_joint_x="-0.07" origin_joint_y="-0.11" />
     <xacro:standoff_rod prefix="lower_left" origin_joint_x="-0.07" origin_joint_y="0.11" />
     <xacro:standoff_rod prefix="upper_left" origin_joint_x="0.07" origin_joint_y="0.11" />
-    <!-- Cup Holder Tray -->
+    <!-- Cup Holder Tray + Joint -->
     <xacro:cup_holder_tray />
     <!-- Include Laser scanner or not -->

File: xacro/caster_wheel.xacro (robot description, xacro)
@@ -1,16 +1,5 @@
 <?xml version="1.0"?>
 <robot xmlns:xacro="http://www.ros.org/wiki/xacro">
-    <!--xacro:property name="caster_wheel_radius" value="0.0352" />
-    <xacro:property name="caster_wheel_mass" value="0.05" />
-    <xacro:property name="negligible_mass" value="0.001" /-->
-    <!-- sphere_inertia"
-    # params="mass r"
-    # mass: Mass in Kilograms of the link
-    # r: Radius of the sphere in meters -->
-    <xacro:macro name="sphere_inertia" params="mass r" >
-        <inertia ixx="${2*mass*r*r/5}" ixy = "0" ixz = "0"
-                 iyy="${2*mass*r*r/5}" iyz = "0"
-                 izz="${2*mass*r*r/5}" />
-    </xacro:macro>
+    <xacro:include filename="$(find barista_robot_description)/xacro/inertia_macros.xacro" />
     <xacro:macro name="caster_wheel" params="prefix joint_origin_x">
         <!-- Caster wheel -->

File: xacro/cup_holder_tray.xacro (robot description, xacro)
@@ -1,14 +1,5 @@
 <?xml version="1.0"?>
 <robot xmlns:xacro="http://www.ros.org/wiki/xacro">
-    <!-- "cylinder_inertia"
-    # params="mass r l"
-    # mass: Mass in Kilograms of the link
-    # r: Radius of the cylinder in meters
-    # l: height of the cylinder in meters-->
-    <xacro:macro name="cylinder_inertia" params="mass r l" >
-        <inertia ixx="${mass*(3*r*r+l*l)/12}" ixy = "0" ixz = "0"
-                 iyy="${mass*(3*r*r+l*l)/12}" iyz = "0"
-                 izz="${mass*(r*r)/2}" />
-    </xacro:macro>
+    <xacro:include filename="$(find barista_robot_description)/xacro/inertia_macros.xacro" />
     <xacro:macro name="cup_holder_tray">
         <!-- Cup Holder Tray -->

File: xacro/drive_wheel.xacro (robot description, xacro)
@@ -1,14 +1,5 @@
 <?xml version="1.0"?>
 <robot xmlns:xacro="http://www.ros.org/wiki/xacro">
-    <!-- "cylinder_inertia"
-    # params="mass r l"
-    # mass: Mass in Kilograms of the link
-    # r: Radius of the cylinder in meters
-    # l: height of the cylinder in meters-->
-    <xacro:macro name="cylinder_inertia" params="mass r l" >
-        <inertia ixx="${mass*(3*r*r+l*l)/12}" ixy = "0" ixz = "0"
-                 iyy="${mass*(3*r*r+l*l)/12}" iyz = "0"
-                 izz="${mass*(r*r)/2}" />
-    </xacro:macro>
+    <xacro:include filename="$(find barista_robot_description)/xacro/inertia_macros.xacro" />
     <xacro:macro name="drive_wheel" params="drive_wheel_name origin_joint_y">
         <!-- Drive Wheel -->

File: xacro/laser_scanner.xacro (robot description, xacro)
@@ -1,13 +1,5 @@
 <?xml version="1.0"?>
 <robot xmlns:xacro="http://www.ros.org/wiki/xacro">
-    <!-- "box_inertia"
-    # params="mass x y z"
-    # mass: Mass in Kilograms of the link
-    # x,y,z: Are the size of each side of the box in each of the axes in meters -->
-    <xacro:macro name="box_inertia" params="mass x y z" >
-        <inertia ixx="${mass*(y*y+z*z)/12}" ixy = "0" ixz = "0"
-                 iyy="${mass*(x*x+z*z)/12}" iyz = "0"
-                 izz="${mass*(x*x+z*z)/12}" />
-    </xacro:macro>
+    <xacro:include filename="$(find barista_robot_description)/xacro/inertia_macros.xacro" />
     <xacro:macro name="laser_scanner">
         <!-- Laser Scan (Model) -->

File: xacro/standoff_rod.xacro (robot description, xacro)
@@ -1,14 +1,5 @@
 <?xml version="1.0"?>
 <robot xmlns:xacro="http://www.ros.org/wiki/xacro">
-    <!-- "cylinder_inertia"
-    # params="mass r l"
-    # mass: Mass in Kilograms of the link
-    # r: Radius of the cylinder in meters
-    # l: height of the cylinder in meters-->
-    <xacro:macro name="cylinder_inertia" params="mass r l" >
-        <inertia ixx="${mass*(3*r*r+l*l)/12}" ixy = "0" ixz = "0"
-                 iyy="${mass*(3*r*r+l*l)/12}" iyz = "0"
-                 izz="${mass*(r*r)/2}" />
-    </xacro:macro>
+    <xacro:include filename="$(find barista_robot_description)/xacro/inertia_macros.xacro" />
     <xacro:macro name="standoff_rod" params="prefix origin_joint_x origin_joint_y">
         <!-- Standoff rod -->
