Commit message: base_footprint link added to xacro file to move the robot above the ground

File: xacro/barista_robot_model.gazebo_plugins.xacro (robot description, xacro)
@@ -71,5 +71,5 @@
                 <publish_odom_tf>true</publish_odom_tf>
                 <odometry_frame>odom</odometry_frame>
-                <robot_base_frame>base_link</robot_base_frame>
+                <robot_base_frame>base_footprint</robot_base_frame>
             </plugin>
         </gazebo>

File: xacro/barista_robot_model.urdf.xacro (robot description, xacro)
@@ -21,4 +21,11 @@
         <color rgba="0.0 0.5 0.0 1"/>
     </material>
+    <!-- Base Footprint -->
+    <link name="base_footprint"/>
+    <joint name="base_footprint_to_base_link" type="fixed">
+        <origin rpy="0 0 0" xyz="0 0 0.1127" />
+        <parent link="base_footprint"/>
+        <child link="base_link"/>
+    </joint>
     <!-- Base Link -->
     <link name="base_link">

Commit message: Namespace added to Gazebo plugins using argument robot_name defined from xacro command

File: xacro/barista_robot_model.gazebo_plugins.xacro (robot description, xacro)
@@ -6,4 +6,5 @@
             <plugin name="barista_robot_joint_state" filename="libgazebo_ros_joint_state_publisher.so">
                 <ros>
+                    <namespace>${robot_name}</namespace>
                     <remapping>~/out:=joint_states</remapping>
                 </ros>
@@ -43,8 +44,9 @@
                     <plugin name="laser" filename="libgazebo_ros_ray_sensor.so">
                         <ros>
+                            <namespace>${robot_name}</namespace>
                             <remapping>~/out:=scan</remapping>
                         </ros>
                         <output_type>sensor_msgs/LaserScan</output_type>
-                        <frame_name>laser_scan_frame</frame_name>
+                        <frame_name>${robot_name}/laser_scan_frame</frame_name>
                     </plugin>
                 </sensor>
@@ -55,6 +57,7 @@
             <plugin filename="libgazebo_ros_diff_drive.so" name="differential_drive_controller">
                 <ros>
-                    <remapping>cmd_vel:=/cmd_vel</remapping>
-                    <remapping>odom:=/odom</remapping>
+                    <namespace>${robot_name}</namespace>
+                    <remapping>/cmd_vel:=cmd_vel</remapping>
+                    <remapping>/odom:=odom</remapping>
                 </ros>
                 <!-- wheel joints -->
@@ -70,6 +73,6 @@
                 <publish_odom>true</publish_odom>
                 <publish_odom_tf>true</publish_odom_tf>
-                <odometry_frame>odom</odometry_frame>
-                <robot_base_frame>base_footprint</robot_base_frame>
+                <odometry_frame>${robot_name}/odom</odometry_frame>
+                <robot_base_frame>${robot_name}/base_footprint</robot_base_frame>
             </plugin>
         </gazebo>

File: xacro/barista_robot_model.urdf.xacro (robot description, xacro)
@@ -1,4 +1,6 @@
 <?xml version="1.0"?>
 <robot xmlns:xacro="http://www.ros.org/wiki/xacro" name="barista_robot">
+    <!-- Robot name -->
+    <xacro:property name="robot_name" value="$(arg robot_name)" />
     <!-- Robot global dimensions -->
     <xacro:property name="base_link_radius" value="0.178" />
