Commit message: Caster wheels added to xacro file + Caster wheel joints added to joint_state_publisher Gazebo plugin

File: xacro/barista_robot_model.gazebo.xacro (robot description, xacro)
@@ -22,4 +22,20 @@
             <mu2>1.0</mu2>
         </gazebo>
+        <!-- Gazebo - Front Caster Wheel -->
+        <gazebo reference="front_caster_wheel_yaw_link">
+            <material>Gazebo/Green</material>
+            <kp>1000000.0</kp>
+            <kd>100.0</kd>
+            <mu1>0.5</mu1>
+            <mu2>0.5</mu2>
+        </gazebo>
+        <!-- Gazebo - Back Caster Wheel -->
+        <gazebo reference="back_caster_wheel_yaw_link">
+            <material>Gazebo/Green</material>
+            <kp>1000000.0</kp>
+            <kd>100.0</kd>
+            <mu1>0.5</mu1>
+            <mu2>0.5</mu2>
+        </gazebo>
     </xacro:macro>
 </robot>

File: xacro/barista_robot_model.gazebo_plugins.xacro (robot description, xacro)
@@ -11,4 +11,10 @@
                 <joint_name>base_link_to_left_drive_wheel_joint</joint_name>
                 <joint_name>base_link_to_right_drive_wheel_joint</joint_name>
+                <joint_name>front_caster_wheel_roll_joint</joint_name>
+                <joint_name>front_caster_wheel_pitch_joint</joint_name>
+                <joint_name>front_caster_wheel_yaw_joint</joint_name>
+                <joint_name>back_caster_wheel_roll_joint</joint_name>
+                <joint_name>back_caster_wheel_pitch_joint</joint_name>
+                <joint_name>back_caster_wheel_yaw_joint</joint_name>
             </plugin>
         </gazebo>

File: xacro/barista_robot_model.urdf.xacro (robot description, xacro)
@@ -4,4 +4,5 @@
     <xacro:include filename="$(find barista_robot_description)/xacro/barista_robot_model.gazebo_plugins.xacro" />
     <xacro:include filename="$(find barista_robot_description)/xacro/drive_wheel.xacro" />
+    <xacro:include filename="$(find barista_robot_description)/xacro/caster_wheel.xacro" />
     <!-- Colors -->
     <material name="blue">
@@ -51,4 +52,43 @@
         <axis xyz="0 1 0" />
     </joint>
+    <!-- Caster Wheels -->
+    <xacro:caster_wheel prefix="front" />
+    <xacro:caster_wheel prefix="back" />
+    <joint name="front_caster_wheel_roll_joint" type="continuous" >
+        <origin rpy="0 0 0" xyz="0.11 0 -0.0775" />
+        <parent link="base_link" />
+        <child link="front_caster_wheel_roll_link" />
+        <axis xyz="1 0 0" />
+    </joint>
+    <joint name="front_caster_wheel_pitch_joint" type="continuous" >
+        <origin rpy="0 0 0" xyz="0 0 0" />
+        <parent link="front_caster_wheel_roll_link" />
+        <child link="front_caster_wheel_pitch_link" />
+        <axis xyz="0 1 0" />
+    </joint>
+    <joint name="front_caster_wheel_yaw_joint" type="continuous" >
+        <origin rpy="0 0 0" xyz="0 0 0" />
+        <parent link="front_caster_wheel_pitch_link" />
+        <child link="front_caster_wheel_yaw_link" />
+        <axis xyz="0 0 1" />
+    </joint>
+    <joint name="back_caster_wheel_roll_joint" type="continuous" >
+        <origin rpy="0 0 0" xyz="-0.11 0 -0.0775" />
+        <parent link="base_link" />
+        <child link="back_caster_wheel_roll_link" />
+        <axis xyz="1 0 0" />
+    </joint>
+    <joint name="back_caster_wheel_pitch_joint" type="continuous" >
+        <origin rpy="0 0 0" xyz="0 0 0" />
+        <parent link="back_caster_wheel_roll_link" />
+        <child link="back_caster_wheel_pitch_link" />
+        <axis xyz="0 1 0" />
+    </joint>
+    <joint name="back_caster_wheel_yaw_joint" type="continuous" >
+        <origin rpy="0 0 0" xyz="0 0 0" />
+        <parent link="back_caster_wheel_pitch_link" />
+        <child link="back_caster_wheel_yaw_link" />
+        <axis xyz="0 0 1" />
+    </joint>
     <!-- Gazebo physical properties and colors -->
     <xacro:gazebo_elements />

Commit message: Standoff rods added to xacro file

File: xacro/barista_robot_model.gazebo.xacro (robot description, xacro)
@@ -38,4 +38,20 @@
             <mu2>0.5</mu2>
         </gazebo>
+        <!-- Gazebo Color for Upper Right Rod -->
+        <gazebo reference="upper_right_rod">
+            <material>Gazebo/White</material>
+        </gazebo>
+        <!-- Gazebo Color for Lower Right Rod -->
+        <gazebo reference="lower_right_rod">
+            <material>Gazebo/White</material>
+        </gazebo>
+        <!-- Gazebo Color for Lower Left Rod -->
+        <gazebo reference="lower_left_rod">
+            <material>Gazebo/White</material>
+        </gazebo>
+        <!-- Gazebo Color for Upper Left Rod -->
+        <gazebo reference="upper_left_rod">
+            <material>Gazebo/White</material>
+        </gazebo>
     </xacro:macro>
 </robot>

File: xacro/barista_robot_model.urdf.xacro (robot description, xacro)
@@ -5,4 +5,5 @@
     <xacro:include filename="$(find barista_robot_description)/xacro/drive_wheel.xacro" />
     <xacro:include filename="$(find barista_robot_description)/xacro/caster_wheel.xacro" />
+    <xacro:include filename="$(find barista_robot_description)/xacro/standoff_rod.xacro" />
     <!-- Colors -->
     <material name="blue">
@@ -91,4 +92,29 @@
         <axis xyz="0 0 1" />
     </joint>
+    <!-- Standoff rods -->
+    <xacro:standoff_rod prefix="upper_right" />
+    <xacro:standoff_rod prefix="lower_right" />
+    <xacro:standoff_rod prefix="upper_left" />
+    <xacro:standoff_rod prefix="lower_left" />
+    <joint name="base_link_to_upper_right_rod_joint" type="fixed" >
+        <origin rpy="0 0 0" xyz="0.07 -0.11 0.1875" />
+        <parent link="base_link" />
+        <child link="upper_right_rod" />
+    </joint>
+    <joint name="base_link_to_lower_right_rod_joint" type="fixed" >
+        <origin rpy="0 0 0" xyz="-0.07 -0.11 0.1875" />
+        <parent link="base_link" />
+        <child link="lower_right_rod" />
+    </joint>
+    <joint name="base_link_to_lower_left_rod_joint" type="fixed" >
+        <origin rpy="0 0 0" xyz="-0.07 0.11 0.1875" />
+        <parent link="base_link" />
+        <child link="lower_left_rod" />
+    </joint>
+     <joint name="base_link_to_upper_left_rod_joint" type="fixed" >
+        <origin rpy="0 0 0" xyz="0.07 0.11 0.1875" />
+        <parent link="base_link" />
+        <child link="upper_left_rod" />
+    </joint>
     <!-- Gazebo physical properties and colors -->
     <xacro:gazebo_elements />

Commit message: Cup holder tray added to xacro file

File: xacro/barista_robot_model.gazebo.xacro (robot description, xacro)
@@ -54,4 +54,8 @@
             <material>Gazebo/White</material>
         </gazebo>
+        <!-- Gazebo Color for Cup Holder Tray -->
+        <gazebo reference="cup_holder_tray">
+            <material>Gazebo/Blue</material>
+        </gazebo>
     </xacro:macro>
 </robot>

File: xacro/barista_robot_model.urdf.xacro (robot description, xacro)
@@ -6,4 +6,5 @@
     <xacro:include filename="$(find barista_robot_description)/xacro/caster_wheel.xacro" />
     <xacro:include filename="$(find barista_robot_description)/xacro/standoff_rod.xacro" />
+    <xacro:include filename="$(find barista_robot_description)/xacro/cup_holder_tray.xacro" />
     <!-- Colors -->
     <material name="blue">
@@ -117,4 +118,11 @@
         <child link="upper_left_rod" />
     </joint>
+    <!-- Cup Holder Tray -->
+    <xacro:cup_holder_tray />
+    <joint name="base_link_to_cup_holder_tray_joint" type="fixed">
+        <origin rpy="0 0 0" xyz="0 0 0.3425" />
+        <parent link="base_link" />
+        <child link="cup_holder_tray" />
+    </joint>
     <!-- Gazebo physical properties and colors -->
     <xacro:gazebo_elements />

Commit message: Laser scanner added to xacro file with condition inclusion in the final urdf

File: xacro/barista_robot_model.gazebo.xacro (robot description, xacro)
@@ -58,4 +58,8 @@
             <material>Gazebo/Blue</material>
         </gazebo>
+        <!-- Gazebo Color for Laser Scan Link -->
+        <gazebo reference="laser_scan_link">
+            <material>Gazebo/Grey</material>
+        </gazebo>
     </xacro:macro>
 </robot>

File: xacro/barista_robot_model.urdf.xacro (robot description, xacro)
@@ -7,4 +7,5 @@
     <xacro:include filename="$(find barista_robot_description)/xacro/standoff_rod.xacro" />
     <xacro:include filename="$(find barista_robot_description)/xacro/cup_holder_tray.xacro" />
+    <xacro:include filename="$(find barista_robot_description)/xacro/laser_scanner.xacro" />
     <!-- Colors -->
     <material name="blue">
@@ -125,4 +126,19 @@
         <child link="cup_holder_tray" />
     </joint>
+    <xacro:arg name="include_laser" default="true"/>
+    <xacro:if value="$(arg include_laser)">
+        <!-- Laser scanner (Model link and Frame link) -->
+        <xacro:laser_scanner />
+        <joint name="base_link_to_laser_scan_link_joint" type="fixed">
+            <origin rpy="0 0 0" xyz="0.089 0 0.0775"/>
+            <parent link="base_link" />
+            <child link="laser_scan_link" />
+        </joint>
+        <joint name="laser_scan_link_to_frame_joint" type="fixed" >
+            <origin rpy="0 0 0" xyz="0 0 0.05" />
+            <parent link="laser_scan_link" />
+            <child link="laser_scan_frame" />
+        </joint>
+    </xacro:if>
     <!-- Gazebo physical properties and colors -->
     <xacro:gazebo_elements />

Commit message: Update xacro files to spawn 2 robots with different colors (blue and red)

File: xacro/barista_robot_model.gazebo.xacro (robot description, xacro)
@@ -4,5 +4,10 @@
         <!-- Gazebo Color for Base link-->
         <gazebo reference="base_link">
-            <material>Gazebo/Blue</material>
+            <xacro:if value="${robot_name == 'morty'}">
+                <material>Gazebo/Blue</material>
+            </xacro:if>
+            <xacro:unless value="${robot_name == 'morty'}">
+                <material>Gazebo/Red</material>
+            </xacro:unless>
         </gazebo>
         <!-- Gazebo - Left Drive Wheel -->
@@ -56,5 +61,10 @@
         <!-- Gazebo Color for Cup Holder Tray -->
         <gazebo reference="cup_holder_tray">
-            <material>Gazebo/Blue</material>
+            <xacro:if value="${robot_name == 'morty'}">
+                <material>Gazebo/Blue</material>
+            </xacro:if>
+            <xacro:unless value="${robot_name == 'morty'}">
+                <material>Gazebo/Red</material>
+            </xacro:unless>
         </gazebo>
         <!-- Gazebo Color for Laser Scan Link -->

File: xacro/barista_robot_model.urdf.xacro (robot description, xacro)
@@ -2,5 +2,7 @@
 <robot xmlns:xacro="http://www.ros.org/wiki/xacro" name="barista_robot">
     <!-- Robot name -->
-    <xacro:property name="robot_name" value="$(arg robot_name)" />
+    <xacro:property name="robot_name" value="$(arg robot_name)"/>
+    <xacro:property name="robot_color"
+                    value="${'blue' if robot_name == 'morty' else 'red'}"/>
     <!-- Robot global dimensions -->
     <xacro:property name="base_link_radius" value="0.178" />
@@ -44,4 +46,7 @@
         <color rgba="0.0 0.5 0.0 1"/>
     </material>
+    <material name="red">
+        <color rgba="1 0 0 1"/>
+    </material>
     <!-- Base Footprint -->
     <link name="base_footprint"/>
@@ -57,5 +62,6 @@
                 <cylinder radius="${base_link_radius}" length="${base_link_height}" />
             </geometry>
-            <material name="blue" />
+            <!-- Change link color depending on robot_name -->
+            <material name="${robot_color}" />
         </visual>
         <collision>

File: xacro/cup_holder_tray.xacro (robot description, xacro)
@@ -9,5 +9,6 @@
                     <cylinder radius="${tray_radius}" length="${tray_width}" />
                 </geometry>
-                <material name="blue" />
+                <!-- Change link color depending on robot_name -->
+                <material name="${robot_color}" />
             </visual>
             <collision>
