Commit message: Caster wheels added to urdf file

File: urdf/barista_robot_model.urdf (robot description, URDF)
Before this commit: robot barista_robot, 1 links, 0 joints
Links:
- added link left_caster_wheel; collision cylinder length=0.0206 radius=0.0352; visual cylinder length=0.0206 radius=0.0352
- added link right_caster_wheel; collision cylinder length=0.0206 radius=0.0352; visual cylinder length=0.0206 radius=0.0352
Joints:
- added joint base_link_to_left_caster_wheel_joint: type continuous, parent base_link, child left_caster_wheel, origin xyz=0 0.126 -0.07525 rpy=0 0 0, axis 0 1 0
- added joint base_link_to_right_caster_wheel_joint: type continuous, parent base_link, child right_caster_wheel, origin xyz=0 -0.126 -0.07525 rpy=0 0 0, axis 0 1 0

Commit message: Standoff rods added to urdf file

File: urdf/barista_robot_model.urdf (robot description, URDF)
Before this commit: robot barista_robot, 3 links, 2 joints
Links:
- added link lower_left_rod; collision cylinder length=0.22 radius=0.01; visual cylinder length=0.22 radius=0.01
- added link lower_right_rod; collision cylinder length=0.22 radius=0.01; visual cylinder length=0.22 radius=0.01
- added link upper_left_rod; collision cylinder length=0.22 radius=0.01; visual cylinder length=0.22 radius=0.01
- added link upper_right_rod; collision cylinder length=0.22 radius=0.01; visual cylinder length=0.22 radius=0.01
Joints:
- added joint base_link_to_lower_left_rod_joint: type fixed, parent base_link, child lower_left_rod, origin xyz=-0.089 0.126 0.1875 rpy=0 0 0
- added joint base_link_to_lower_right_rod_joint: type fixed, parent base_link, child lower_right_rod, origin xyz=-0.089 -0.126 0.1875 rpy=0 0 0
- added joint base_link_to_upper_left_rod_joint: type fixed, parent base_link, child upper_left_rod, origin xyz=0.089 0.126 0.1875 rpy=0 0 0
- added joint base_link_to_upper_right_rod_joint: type fixed, parent base_link, child upper_right_rod, origin xyz=0.089 -0.126 0.1875 rpy=0 0 0
- joint base_link_to_left_caster_wheel_joint: origin xyz=0 0.126 -0.07525 rpy=0 0 0 -> xyz=0 0.126 -0.0775 rpy=0 0 0
- joint base_link_to_right_caster_wheel_joint: origin xyz=0 -0.126 -0.07525 rpy=0 0 0 -> xyz=0 -0.126 -0.0775 rpy=0 0 0

Commit message: Cup holder tray added to urdf file + rod position ajusted

File: urdf/barista_robot_model.urdf (robot description, URDF)
Before this commit: robot barista_robot, 7 links, 6 joints
Links:
- added link cup_holder_tray; collision cylinder length=0.090 radius=0.160; visual cylinder length=0.090 radius=0.160
Joints:
- added joint base_link_to_cup_holder_tray_joint: type fixed, parent base_link, child cup_holder_tray, origin xyz=0 0 0.3425 rpy=0 0 0
- joint base_link_to_lower_left_rod_joint: origin xyz=-0.089 0.126 0.1875 rpy=0 0 0 -> xyz=-0.07 0.11 0.1875 rpy=0 0 0
- joint base_link_to_lower_right_rod_joint: origin xyz=-0.089 -0.126 0.1875 rpy=0 0 0 -> xyz=-0.07 -0.11 0.1875 rpy=0 0 0
- joint base_link_to_upper_left_rod_joint: origin xyz=0.089 0.126 0.1875 rpy=0 0 0 -> xyz=0.07 0.11 0.1875 rpy=0 0 0
- joint base_link_to_upper_right_rod_joint: origin xyz=0.089 -0.126 0.1875 rpy=0 0 0 -> xyz=0.07 -0.11 0.1875 rpy=0 0 0

Commit message: Laser scanner added to urdf file

File: urdf/barista_robot_model.urdf (robot description, URDF)
Before this commit: robot barista_robot, 8 links, 7 joints
Links:
- added link laser_scan_frame
- added link laser_scan_link; collision box size=0.02 0.02 0.05; visual mesh filename=file:///home/user/ros2_ws/src/checkpoint4_auxiliary_files/m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
Joints:
- added joint base_link_to_laser_scan_link_joint: type fixed, parent base_link, child laser_scan_link, origin xyz=0.089 0 0.0775 rpy=0 0 0
- added joint laser_scan_link_to_frame_joint: type fixed, parent laser_scan_link, child laser_scan_frame, origin xyz=0 0 0.03 rpy=0 0 0

Commit message: Mesh file for laser scanner added to /meshes

File: urdf/barista_robot_model.urdf (robot description, URDF)
Before this commit: robot barista_robot, 10 links, 9 joints
Links:
- link laser_scan_link: geometry collision box size=0.02 0.02 0.05; visual mesh filename=package://barista_robot_description/meshes/hokuyo_urg_04lx.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

Commit message: Inertial added to all robot links

File: urdf/barista_robot_model.urdf (robot description, URDF)
Before this commit: robot barista_robot, 10 links, 9 joints
Links:
- link base_link: mass None -> 0.5
- link cup_holder_tray: mass None -> 0.25
- link laser_scan_link: mass None -> 0.05
- link left_caster_wheel: mass None -> 0.05
- link lower_left_rod: mass None -> 0.025
- link lower_right_rod: mass None -> 0.025
- link right_caster_wheel: mass None -> 0.05
- link upper_left_rod: mass None -> 0.025
- link upper_right_rod: mass None -> 0.025

Commit message: Fix - Correct wheel link name (from caster to drive)

File: urdf/barista_robot_model.urdf (robot description, URDF)
Before this commit: robot barista_robot, 10 links, 9 joints
Links:
- removed link left_caster_wheel
- removed link right_caster_wheel
- added link left_drive_wheel, mass 0.05; collision cylinder length=0.0206 radius=0.0352; visual cylinder length=0.0206 radius=0.0352
- added link right_drive_wheel, mass 0.05; collision cylinder length=0.0206 radius=0.0352; visual cylinder length=0.0206 radius=0.0352
Joints:
- removed joint base_link_to_left_caster_wheel_joint
- removed joint base_link_to_right_caster_wheel_joint
- added joint base_link_to_left_drive_wheel_joint: type continuous, parent base_link, child left_drive_wheel, origin xyz=0 0.126 -0.0775 rpy=0 0 0, axis 0 1 0
- added joint base_link_to_right_drive_wheel_joint: type continuous, parent base_link, child right_drive_wheel, origin xyz=0 -0.126 -0.0775 rpy=0 0 0, axis 0 1 0

Commit message: Caster wheels added to urdf file (not drive wheels)

File: urdf/barista_robot_model.urdf (robot description, URDF)
Before this commit: robot barista_robot, 10 links, 9 joints
Links:
- added link front_caster_wheel_pitch_link, mass 0.001
- added link front_caster_wheel_roll_link, mass 0.001
- added link front_caster_wheel_yaw_link, mass 0.05; collision sphere radius=0.0352; visual sphere radius=0.0352
Joints:
- added joint front_caster_wheel_pitch_joint: type continuous, parent front_caster_wheel_roll_link, child front_caster_wheel_pitch_link, origin xyz=0 0 0 rpy=0 0 0, axis 0 1 0
- added joint front_caster_wheel_roll_joint: type continuous, parent base_link, child front_caster_wheel_roll_link, origin xyz=0.11 0 -0.0775 rpy=0 0 0, axis 1 0 0
- added joint front_caster_wheel_yaw_joint: type continuous, parent front_caster_wheel_pitch_link, child front_caster_wheel_yaw_link, origin xyz=0 0 0 rpy=0 0 0, axis 0 0 1

Commit message: Back caster wheel added to urdf file

File: urdf/barista_robot_model.urdf (robot description, URDF)
Before this commit: robot barista_robot, 13 links, 12 joints
Links:
- added link back_caster_wheel_pitch_link, mass 0.001
- added link back_caster_wheel_roll_link, mass 0.001
- added link back_caster_wheel_yaw_link, mass 0.05; collision sphere radius=0.0352; visual sphere radius=0.0352
Joints:
- added joint back_caster_wheel_pitch_joint: type continuous, parent back_caster_wheel_roll_link, child back_caster_wheel_pitch_link, origin xyz=0 0 0 rpy=0 0 0, axis 0 1 0
- added joint back_caster_wheel_roll_joint: type continuous, parent base_link, child back_caster_wheel_roll_link, origin xyz=-0.11 0 -0.0775 rpy=0 0 0, axis 1 0 0
- added joint back_caster_wheel_yaw_joint: type continuous, parent back_caster_wheel_pitch_link, child back_caster_wheel_yaw_link, origin xyz=0 0 0 rpy=0 0 0, axis 0 0 1

Commit message: Gazebo Lidar plugin added to urdf file + Moved lidar joint up by 2 cm

File: urdf/barista_robot_model.urdf (robot description, URDF)
Before this commit: robot barista_robot, 16 links, 15 joints
Joints:
- joint laser_scan_link_to_frame_joint: origin xyz=0 0 0.03 rpy=0 0 0 -> xyz=0 0 0.05 rpy=0 0 0

Commit message: base_footprint link added to urdf file to move the robot above the ground + Update RViz configuration to define base_footprint as fixed frame

File: urdf/barista_robot_model.urdf (robot description, URDF)
Before this commit: robot barista_robot, 16 links, 15 joints
Links:
- added link base_footprint
Joints:
- added joint base_footprint_to_base_link: type fixed, parent base_footprint, child base_link, origin xyz=0 0 0.1127 rpy=0 0 0
